Commit message: Added Camera Calibration

File: install/tb3_description/share/tb3_description/urdf/turtlebot3_burger_base.urdf (robot description, URDF)
Before this commit: robot turtlebot3_burger, 5 links, 4 joints
Links:
- added link camera_lens_link
- added link camera_link, mass 0.001; collision mesh filename=file:///home/papasav/robot_ws/install/tb3_description/share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 scale=0.0001 0.0001 0.0001; visual mesh filename=file:///home/papasav/robot_ws/install/tb3_description/share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 scale=0.0001 0.0001 0.0001
- added link laser_link, mass 0.2; collision box size=0.09 0.056 0.073; visual mesh filename=file:///home/papasav/robot_ws/install/tb3_description/share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 scale=0.001 0.001 0.001
- link base_link: geometry collision box size=0.17 0.16 0.16; visual mesh filename=file:///home/papasav/robot_ws/install/tb3_description/share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 scale=0.001 0.001 0.001
- link wheel_left_link: geometry collision cylinder length=0.018 radius=0.033; visual mesh filename=file:///home/papasav/robot_ws/install/tb3_description/share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 scale=0.001 0.001 0.001
- link wheel_right_link: geometry collision cylinder length=0.018 radius=0.033; visual mesh filename=file:///home/papasav/robot_ws/install/tb3_description/share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 scale=0.001 0.001 0.001
Joints:
- added joint camera_base_joint: type fixed, parent base_link, child camera_link, origin xyz=0.065 0.0 0.095 rpy=0 0 0
- added joint camera_lens_joint: type fixed, parent camera_link, child camera_lens_link, origin xyz=0.025 -0.015 0.02 rpy=0 0 0
- added joint laser_joint: type fixed, parent base_link, child laser_link, origin xyz=-0.005 0.0 0.18 rpy=0 0 0

Commit message: Update

File: install/tb3_description/share/tb3_description/urdf/turtlebot3_burger_base.urdf (robot description, URDF)
Before this commit: robot turtlebot3_burger, 8 links, 7 joints
Links:
- link camera_link: geometry collision mesh filename=file:///home/bot12/robot_ws/install/tb3_description/share/t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 scale=0.0001 0.0001 0.0001; visual mesh filename=file:///home/bot12/robot_ws/install/tb3_description/share/t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 scale=0.0001 0.0001 0.0001
- link laser_link: geometry collision box size=0.09 0.056 0.073; visual mesh filename=file:///home/bot12/robot_ws/install/tb3_description/share/t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 scale=0.001 0.001 0.001

File: install/tb3_description/share/tb3_description/urdf/turtlebot3_burger_base.urdf.xacro (robot description, xacro)
@@ -4,6 +4,6 @@
   <xacro:include filename="$(find tb3_description)/urdf/common_properties.xacro"/>
 	<!-- Turtlebot3 platform include files -->
-    <xacro:include filename="$(find tb3_description)/urdf/wheel.urdf.xacro"/>
-    <xacro:include filename="$(find tb3_description)/urdf/caster.urdf.xacro"/>
+  <xacro:include filename="$(find tb3_description)/urdf/wheel.urdf.xacro"/>
+  <xacro:include filename="$(find tb3_description)/urdf/caster.urdf.xacro"/>
 	<!-- Base -->
   <link name="base_link">
@@ -23,11 +23,11 @@
   </link>
   <link name="base_footprint">
-      <inertial>
-      <origin xyz="0.0 0.0 0.0125" rpy="0 0 0"/>
-      <mass value="1.5"/>
-      <inertia ixx="0.0270833333" ixy="0.0" ixz="0.0"
-               iyy="0.01215" iyz="0.0"
-               izz="0.0270833333" />
-      </inertial>
+    <inertial>
+    <origin xyz="0.0 0.0 0.0125" rpy="0 0 0"/>
+    <mass value="1.5"/>
+    <inertia ixx="0.0270833333" ixy="0.0" ixz="0.0"
+              iyy="0.01215" iyz="0.0"
+              izz="0.0270833333" />
+    </inertial>
   </link>
   <joint name="base_joint" type="fixed">
@@ -37,17 +37,17 @@
   </joint>
 	<!-- Turtlebot3 wheel macros -->
-    <xacro:turtlebot3_wheel alignment="left">
-        <origin xyz="0.0375 0.075 0.018" rpy="0 0 0"/>
-    </xacro:turtlebot3_wheel>
-    <xacro:turtlebot3_wheel alignment="right">
-        <origin xyz="0.0375 -0.075 0.018" rpy="0 0 0"/>
-    </xacro:turtlebot3_wheel>
+  <xacro:turtlebot3_wheel alignment="left">
+    <origin xyz="0.0375 0.075 0.018" rpy="0 0 0"/>
+  </xacro:turtlebot3_wheel>
+  <xacro:turtlebot3_wheel alignment="right">
+    <origin xyz="0.0375 -0.075 0.018" rpy="0 0 0"/>
+  </xacro:turtlebot3_wheel>
 	<!-- Turtlebot3 caster macros -->
-    <xacro:turtlebot3_caster alignment="center">
-        <origin xyz="-0.04 0.0 0.0" rpy="0 0 0"/>
-    </xacro:turtlebot3_caster>
-    <!-- Sensors -->
-    <xacro:include filename="$(find tb3_description)/urdf/camera.urdf.xacro"/>
-    <xacro:include filename="$(find tb3_description)/urdf/laser.urdf.xacro"/>
+  <xacro:turtlebot3_caster alignment="center">
+    <origin xyz="-0.04 0.0 0.0" rpy="0 0 0"/>
+  </xacro:turtlebot3_caster>
+  <!-- Sensors -->
+  <xacro:include filename="$(find tb3_description)/urdf/camera.urdf.xacro"/>
+  <xacro:include filename="$(find tb3_description)/urdf/laser.urdf.xacro"/>
   <!-- Plugins -->
 </robot>

Commit message: April Tag

File: install/tb3_description/share/tb3_description/urdf/turtlebot3_burger_base.urdf (robot description, URDF)
Before this commit: robot turtlebot3_burger, 8 links, 7 joints
Links:
- link base_link: geometry collision box size=0.17 0.16 0.16; visual mesh filename=file:///home/bot12/robot_ws/install/tb3_description/share/t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 scale=0.001 0.001 0.001
- link wheel_left_link: geometry collision cylinder length=0.018 radius=0.033; visual mesh filename=file:///home/bot12/robot_ws/install/tb3_description/share/t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 scale=0.001 0.001 0.001
- link wheel_right_link: geometry collision cylinder length=0.018 radius=0.033; visual mesh filename=file:///home/bot12/robot_ws/install/tb3_description/share/t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 scale=0.001 0.001 0.001

Commit message: AprilTags Detection

File: install/tb3_description/share/tb3_description/urdf/turtlebot3_burger_base.urdf (robot description, URDF)
Before this commit: robot turtlebot3_burger, 8 links, 7 joints
Links:
- link base_link: geometry collision box size=0.17 0.16 0.16; visual mesh filename=file:///home/papasav/robot_ws/install/tb3_description/share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 scale=0.001 0.001 0.001
- link camera_link: geometry collision mesh filename=file:///home/papasav/robot_ws/install/tb3_description/share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 scale=0.0001 0.0001 0.0001; visual mesh filename=file:///home/papasav/robot_ws/install/tb3_description/share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 scale=0.0001 0.0001 0.0001
- link laser_link: geometry collision box size=0.09 0.056 0.073; visual mesh filename=file:///home/papasav/robot_ws/install/tb3_description/share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 scale=0.001 0.001 0.001
- link wheel_left_link: geometry collision cylinder length=0.018 radius=0.033; visual mesh filename=file:///home/papasav/robot_ws/install/tb3_description/share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 scale=0.001 0.001 0.001
- link wheel_right_link: geometry collision cylinder length=0.018 radius=0.033; visual mesh filename=file:///home/papasav/robot_ws/install/tb3_description/share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 scale=0.001 0.001 0.001
